File: MeasureBoard.kicad_pcb (KiCad board)
At the start: 2 copper layers, 60 x 80 mm, 130 parts, among them J1 Conn_01x06, J10 Conn_02x05_Odd_Even, J11 Conn_01x06, J12 Conn_01x06, J13 GS3, J14 USB_OTG, J15 Conn_01x02, J16 Conn_01x03, J17 Conn_01x02, J18 Conn_01x03, J19 Conn_01x03, J2 Conn_01x04, J20 Conn_01x03, J21 Conn_01x03, J22 Conn_01x03, J23 Conn_01x03, J24 Conn_02x05_Odd_Even, J3 GS3, J4 GS2, J5 Conn_01x04, J6 Conn_01x03, J7 Conn_01x04, J8 BARREL_JACK, J9 CONN_01X02, SW1 DIP_SW_2P, SW2 SKRPACE010, SW3 SKRPACE010, SW4 SKRPACE010, U1 L7805, U2 AP1117-33, U3 STM32F103CBTx, U4 NC7SZ08, U5 SP3481CN, U6 NC7WZ241, U7 LTC2875-S8, U8 AM26LV32, Y1 Crystal

Commit message: update
Parts:
- R18: moved to F.Cu
- moved D9 34.7 mm to (91.1, 81.0)
- moved R16 34.7 mm to (91.1, 79.5)
- moved D7 4.44 mm to (70.9, 122.2), turned to 90 degrees
- moved C28 2.80 mm to (68.4, 123.1)
- moved C30 2.40 mm to (68.4, 120.5)
- moved J10 2.28 mm to (76.2, 112.3), turned to 270 degrees
- moved D11 2.00 mm to (57.4, 95.1)
- moved F1 2.00 mm to (58.2, 92.7)
- moved J14 2.00 mm to (52.8, 95.0)
- moved R19 2.00 mm to (58.2, 96.8)
- moved R20 2.00 mm to (58.2, 95.4)
- moved R21 2.00 mm to (58.2, 94.0)
- moved R18 1.86 mm to (81.0, 114.2), turned to 0 degrees
- moved L1 0.50 mm to (86.5, 122.9)
- moved RN2 0.28 mm to (68.2, 121.4)
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Routing:
- net /USB/D-: track 0.00 -> 37.4 mm, vias 0 -> 1
- net /USB/D+: track 0.00 -> 33.0 mm, vias 0 -> 1
- net GND: track 218.6 -> 247.6 mm, vias 23 -> 32
- net /MCU/I2C1_SCL: track 0.00 -> 26.3 mm
- net /MCU/I2C1_SDA: track 0.00 -> 24.4 mm
- net +3V3: track 126.0 -> 143.8 mm, vias 6 -> 7
- net +5V: track 60.9 -> 67.7 mm
- net +12V: track 57.9 -> 64.4 mm
- net /IN_Di/DI2_LPF: track 0.75 -> 6.56 mm
- net NRST: track 23.9 -> 28.8 mm, vias 3 -> 4
- net /IN_Di/DI3_LPF: track 0.79 -> 5.42 mm, vias 1 -> 0
- net /MCU/SYS_JTDI: track 0.00 -> 4.42 mm, vias 0 -> 1
- net /JTAG/SWO-TDO: track 8.35 -> 3.99 mm, vias 0 -> 1
- net /JTAG/SWCLK-TCK: track 8.46 -> 5.51 mm, vias 2 -> 1
- net Net-(J2-Pad1): track 0.00 -> 2.70 mm
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
Commit message: update
Parts:
- C4, C6: footprint Capacitors_SMD:C_0805 -> Capacitors_SMD:C_1206
- U1: footprint TO_SOT_Packages_THT:TO-220-3_Horizontal -> TO_SOT_Packages_THT:TO-220-3_Horizontal_Reversed
- moved C6 4.81 mm to (90.6, 89.8)
- moved U1 4.78 mm to (85.3, 87.5), turned to 0 degrees
- moved D8 2.10 mm to (92.0, 94.5)
- moved C7 1.00 mm to (85.6, 89.8)
- moved C4 0.82 mm to (86.4, 85.2)
- moved U2 0.20 mm to (85.6, 94.6)
Connections:
- U3 pad 28: /IN_Di/DI3_LPF -> /IN_Di/DI1_LPF
- U3 pad 40: /IN_Di/DI1_LPF -> /IN_Di/DI3_LPF
Routing:
- net +3V3: track 143.8 -> 156.6 mm
- net GND: track 247.6 -> 259.9 mm
- net Net-(C6-Pad1): track 0.00 -> 6.48 mm
- net /IN_Di/DI3_LPF: track 5.42 -> 0.07 mm
- net +5V: track 67.7 -> 71.1 mm
- net Net-(J1-Pad6): track 0.00 -> 2.69 mm
- net +12V: track 64.4 -> 66.7 mm

Commit message: update
Parts:
- removed J16: Conn_01x03, Pin_Headers:Pin_Header_Straight_1x03_Pitch2.54mm
- removed REF** (x4): MountingHole_3.2mm_M3, Mounting_Holes:MountingHole_3.2mm_M3
- removed REF**: Molex_SPOX-5267_22-03-5035_03x2.54mm_Straight, Connectors_Molex:Molex_SPOX-5267_22-03-5035_03x2.54mm_Straight
- added J25: TEST_1P, Mounting_Holes:MountingHole_3.2mm_M3_Pad, F.Cu at (54.0, 146.0)
- added J26: TEST_1P, Mounting_Holes:MountingHole_3.2mm_M3_Pad, F.Cu at (106.0, 146.0)
- added J27: TEST_1P, Mounting_Holes:MountingHole_3.2mm_M3_Pad, F.Cu at (54.0, 74.0)
- added J28: TEST_1P, Mounting_Holes:MountingHole_3.2mm_M3_Pad, F.Cu at (106.0, 74.0)
- added R30: R, Resistors_SMD:R_0603, B.Cu at (102.0, 115.6)
- J11: value Conn_01x06 -> Conn_01x04; footprint Connectors_JST:JST_SH_BM06B-SRSS-TB_06x1.00mm_Straight -> Pin_Headers:Pin_Header_Angled_1x04_Pitch2.54mm
- R16: moved to B.Cu
- moved D9 22.6 mm to (96.0, 103.0)
- moved R16 22.4 mm to (94.2, 101.6), turned to 90 degrees
- moved J11 15.9 mm to (69.8, 87.8), turned to 90 degrees
- moved D5 12.0 mm to (69.0, 94.8), turned to 180 degrees
- moved J17 10.8 mm to (96.5, 116.2)
- moved C1 9.26 mm to (69.8, 92.3), turned to 180 degrees
- moved R26 9.18 mm to (105.0, 115.6)
- moved R2 3.74 mm to (81.0, 82.6)
- moved R1 3.23 mm to (82.6, 82.6)
- moved C5 2.48 mm to (87.8, 99.2)
- moved F1 2.20 mm to (58.2, 90.5)
- moved J14 2.20 mm to (52.8, 92.8)
- moved R19 2.20 mm to (58.2, 94.6)
- moved R20 2.20 mm to (58.2, 93.2)
- moved R21 2.20 mm to (58.2, 91.8)
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Connections:
- J11 pad 1: +3V3 -> Net-(D5-Pad2)
- J11 pad 2: /JTAG/SWCLK-TCK -> GND
- J11 pad 3: GND -> /MCU/USART1_RX
- J11 pad 4: /JTAG/SWDIO-TMS -> /MCU/USART1_TX
- R1 pad 2: Net-(D1-Pad4) -> Net-(D1-Pad2)
- R2 pad 2: Net-(D1-Pad2) -> Net-(D1-Pad4)
- RN2 pad 1: /IN_Di/DI1_LPF -> Net-(RN2-Pad1)
- RN2 pad 2: /IN_Di/DI2_LPF -> /IN_Di/DI3_LPF
- RN2 pad 3: /IN_Di/DI3_LPF -> /IN_Di/DI2_LPF
- RN2 pad 4: Net-(RN2-Pad4) -> /IN_Di/DI1_LPF
- RN2 pad 5: Net-(RN2-Pad5) -> Net-(J23-Pad3)
- RN2 pad 6: Net-(J23-Pad3) -> Net-(J22-Pad3)
- RN2 pad 7: Net-(J22-Pad3) -> Net-(J21-Pad3)
- RN2 pad 8: Net-(J21-Pad3) -> Net-(RN2-Pad8)
- U3 pad 28: /IN_Di/DI1_LPF -> /IN_Di/DI3_LPF
- U3 pad 40: /IN_Di/DI3_LPF -> /IN_Di/DI1_LPF
Routing:
- net GND: track 259.9 -> 340.4 mm, vias 32 -> 38
- net /MCU/USART1_RX: track 1.35 -> 48.4 mm, vias 1 -> 2
- net /MCU/USART1_TX: track 1.35 -> 46.6 mm, vias 1 -> 2
- net +3V3: track 156.6 -> 193.3 mm, vias 7 -> 13
- net Net-(J23-Pad3): track 0.00 -> 16.2 mm
- net Net-(J22-Pad3): track 0.00 -> 12.0 mm
- net +5V: track 71.1 -> 82.4 mm, vias 2 -> 3
- net /MCU/CAN_RX: track 11.3 -> 22.1 mm
- net Net-(J21-Pad3): track 0.00 -> 9.08 mm
- net /MCU/CAN_TX: track 10.5 -> 19.0 mm
- net Net-(D5-Pad2): track 0.00 -> 8.15 mm
- net /IN_Di/DI3_LPF: track 0.07 -> 6.97 mm, vias 0 -> 1
- net NRST: track 28.8 -> 33.9 mm
- net Net-(D11-Pad2): track 0.00 -> 3.84 mm, vias 0 -> 1
- net Net-(R30-Pad2): track 5.49 -> 1.80 mm
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Other:
- outline, holes or cut-outs redrawn
- board text added: "Analog"
- board text added: "Board"
- board text added: "Digital"
- board text added: "F103"
- board text added: "F303"
- board text added: "I2C"
- board text added: "Measurement"
- board text removed: "Ain"
- board text removed: "Din"
- board text removed: "Normal"
- board text removed: "SWD"
- board text removed: "Sandby"
- board text removed: "VCC (3V3,5V)"

Commit message: update
Parts:
- D10: moved to F.Cu
- moved D10 37.6 mm to (77.1, 104.6), turned to 0 degrees
- moved R17 34.7 mm to (77.9, 105.3)
- moved R16 7.65 mm to (97.5, 108.5), turned to 0 degrees
- moved J3 3.70 mm to (51.8, 107.2)
- moved D9 3.50 mm to (96.0, 106.5), turned to 270 degrees
- moved C8 1.75 mm to (90.4, 120.3)
- moved Y1 1.60 mm to (90.4, 122.9)
- moved R14 1.60 mm to (98.5, 125.3)
- moved R15 1.58 mm to (98.5, 121.6)
- moved C9 1.45 mm to (90.4, 125.5)
- moved R13 1.30 mm to (95.2, 121.6)
- moved R12 1.28 mm to (95.2, 125.4)
- moved C2 1.23 mm to (96.6, 125.3)
- moved C3 1.21 mm to (96.6, 121.6)
Connections:
- J14 pad 5: GNDPWR -> GND
- J14 pad 6: GNDPWR -> GND
- R10 pad 2: /MCU/PC14 -> /MCU/PC15
- R11 pad 2: /MCU/PC15 -> /MCU/PC14
- R19 pad 2: GNDPWR -> GND
- SW1 pad 1: /MCU/PC14 -> /MCU/PC15
- SW1 pad 2: /MCU/PC15 -> /MCU/PC14
Routing:
- net +5V: track 82.4 -> 169.3 mm, vias 3 -> 8
- net GND: track 340.4 -> 386.9 mm, vias 38 -> 52
- net /MCU/PC15: track 4.08 -> 18.2 mm
- net /MCU/PC14: track 2.99 -> 16.4 mm
- net /IN_Di/DI1_LPF: track 3.08 -> 14.3 mm, vias 2 -> 3
- net +3V3: track 193.3 -> 186.5 mm, vias 13 -> 14
- net Net-(J2-Pad1): track 2.70 -> 5.36 mm
- net Net-(R13-Pad1): track 1.86 -> 3.70 mm
- net Net-(R12-Pad1): track 1.79 -> 3.46 mm
- net Net-(D10-Pad2): track 0.00 -> 1.55 mm, vias 0 -> 1
- net Net-(C9-Pad2): track 9.60 -> 10.7 mm
- net +12V: track 66.7 -> 66.0 mm
Other:
- board text added: "Designed"
- board text added: "Encoder(ABI)"
- board text added: "by @yuqlid"
- board text added: "v1.0"
- board text removed: "Diff_Encoder(ABI)"

Commit message: update
Parts:
- moved R6 5.43 mm to (59.4, 106.0), turned to 0 degrees
- moved R7 5.41 mm to (62.0, 106.0), turned to 180 degrees
Routing:
- net +3V3: track 186.5 -> 275.4 mm, vias 14 -> 17
- net GND: track 386.9 -> 370.6 mm, vias 52 -> 54
- net /MCU/PC13: track 3.52 -> 18.2 mm, vias 1 -> 2
- net +5V: track 169.3 -> 182.3 mm, vias 8 -> 6
- net /MCU/I2C1_SDA: track 26.7 -> 29.5 mm
- net /MCU/USART1_RX: track 48.4 -> 46.8 mm, vias 2 -> 1
- net /USB/D-: track 38.8 -> 37.7 mm
- net /IN_Di/DI1_LPF: track 14.3 -> 15.3 mm
- net /MCU/I2C1_SCL: track 28.7 -> 29.2 mm
- net /MCU/USART1_TX: vias 2 -> 1

Commit message: update
Parts:
- moved D6 6.04 mm to (94.3, 130.6)
- moved C8 2.73 mm to (92.9, 121.4), turned to 270 degrees
- moved C9 2.73 mm to (92.9, 124.4), turned to 90 degrees
- moved C2 2.60 mm to (99.1, 124.6), turned to 180 degrees
- moved C3 2.51 mm to (99.1, 121.8), turned to 180 degrees
- moved R15 1.71 mm to (99.1, 123.2), turned to 180 degrees
- moved R13 1.53 mm to (96.5, 122.4)
- moved R12 1.32 mm to (96.5, 125.2)
- moved R14 0.92 mm to (99.1, 126.0), turned to 180 degrees
- moved C10 0.50 mm to (86.1, 118.5)
- moved C11 0.50 mm to (84.8, 118.5)
Connections:
- C2 pad 2: /MCU/PB5 -> /MCU/PC15
- C3 pad 2: /MCU/PC13 -> /MCU/PC14
- R10 pad 2: /MCU/PC15 -> /MCU/PC13
- R11 pad 2: /MCU/PC14 -> /MCU/PB5
- R12 pad 2: /MCU/PB5 -> /MCU/PC15
- R13 pad 2: /MCU/PC13 -> /MCU/PC14
- SW1 pad 1: /MCU/PC15 -> /MCU/PC13
- SW1 pad 2: /MCU/PC14 -> /MCU/PB5
Routing:
- net GND: track 370.6 -> 514.0 mm
- net /MCU/PB5: track 3.42 -> 21.8 mm
- net +12V: track 66.0 -> 79.5 mm
- net Net-(D6-Pad2): track 7.34 -> 2.15 mm
- net Net-(D6-Pad4): track 10.0 -> 4.96 mm
- net NRST: track 33.9 -> 30.4 mm
- net +3V3: track 275.4 -> 278.5 mm, vias 17 -> 18
- net /MCU/PC13: track 18.2 -> 20.4 mm, vias 2 -> 1
- net /MCU/PC15: track 18.2 -> 19.7 mm, vias 1 -> 0
- net /JTAG/SWDIO-TMS: track 10.1 -> 8.71 mm
- net /MCU/PC14: track 16.4 -> 17.1 mm, vias 1 -> 0
- net Net-(R12-Pad1): track 3.46 -> 4.13 mm
- net Net-(C8-Pad2): track 9.48 -> 10.1 mm
- net Net-(C9-Pad2): track 10.7 -> 11.3 mm
- net /MCU/USART1_TX: track 46.6 -> 47.3 mm
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
Commit message: update
Parts:
- moved R11 1.10 mm to (90.3, 111.9)
- moved R10 1.05 mm to (91.8, 111.9)
Routing:
- net GND: track 514.0 -> 549.7 mm, vias 54 -> 71
- net +3V3: track 278.5 -> 284.6 mm, vias 18 -> 17
- net /MCU/PC13: track 20.4 -> 22.4 mm
- net /MCU/PB5: track 21.8 -> 22.6 mm
- net /MCU/USART1_TX: track 47.3 -> 47.9 mm

Commit message: update
Routing:
- net GND: track 549.7 -> 673.7 mm, vias 71 -> 119
- net +5V: track 182.4 -> 183.6 mm
- net /MCU/PC13: track 22.4 -> 23.5 mm
- net /MCU/PB5: track 22.6 -> 23.7 mm
- net +3V3: track 284.6 -> 285.7 mm
